File: parte de carga.sch (EAGLE design)
At the start: 42 parts, among them IC1 MCP73831T-2ACI_OT, IC10 741G3157DBVR, IC15 LMV321AIDCKR, IC16 LMV321AIDCKR, IC2 ESP32-S3-WROOM-1-N16R2, IC3 LMV321AIDCKR, IC5 LMV321AIDCKR, IC7 AD8226ARZ, IC9 LP38692MP-3.3_NOPB, J1 USB3500-30-A-KIT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

Commit message: acomode los compenentes dentro de la placa falta organizarlos y elimine una parte de los filtros que no estaba amplificando nada
Parts:
- removed C1: 0.47uF, GCM21B5C2A393JE02L:GCM21B5C2A393JE02L
- removed C3: 0.1uF, GCM21B5C2A393JE02L:GCM21B5C2A393JE02L
- removed IC3: LMV321AIDCKR, LMV321AIDCKR:LMV321AIDCKR
- removed R1: 5.6K, rcl:R-EU_R0805
- removed R6: 10K, rcl:R-EU_R0805
Connections:
- removed net N$16: C1.1, IC3.-IN, IC3.OUT
- removed net N$20: R1.2, R6.1
- removed net N$7: C1.2, C3.2, IC3.+IN, R6.2
- net +3V3: no longer IC3.V+
- net GND: no longer IC3.V-
- net N$8: no longer R1.1
- net VOUT1: now also C5.1
- net VSS: no longer C3.1
Changed lines of the file:
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@@
 <setting verticaltext="up"/>
 </settings>
-<grid distance="0.1" unitdist="inch" unit="inch" style="dots" multiple="1" display="no" altdistance="0.01" altunitdist="inch" altunit="inch"/>
+<grid distance="0.1" unitdist="inch" unit="inch" style="lines" multiple="1" display="no" altdistance="0.01" altunitdist="inch" altunit="inch"/>
 <layers>
 <layer number="1" name="Top" color="4" fill="1" visible="yes" active="no"/>
@@
 <part name="SV2" library="con-lstb" library_urn="urn:adsk.eagle:library:162" deviceset="MA03-1" device="" package3d_urn="urn:adsk.eagle:package:8339/1"/>
 <part name="GND19" library="supply1" library_urn="urn:adsk.eagle:library:371" deviceset="GND" device=""/>
-<part name="IC3" library="LMV321AIDCKR" deviceset="LMV321AIDCKR" device=""/>
-<part name="R1" library="rcl" library_urn="urn:adsk.eagle:library:334" deviceset="R-EU_" device="R0805" package3d_urn="urn:adsk.eagle:package:23553/2" value="5.6K"/>
-<part name="R6" library="rcl" library_urn="urn:adsk.eagle:library:334" deviceset="R-EU_" device="R0805" package3d_urn="urn:adsk.eagle:package:23553/2" value="10K"/>
-<part name="C1" library="GCM21B5C2A393JE02L" deviceset="GCM21B5C2A393JE02L" device="" value="0.47uF"/>
 <part name="GND20" library="supply1" library_urn="urn:adsk.eagle:library:371" deviceset="GND" device=""/>
-<part name="GND21" library="supply1" library_urn="urn:adsk.eagle:library:371" deviceset="GND" device=""/>
-<part name="C3" library="GCM21B5C2A393JE02L" deviceset="GCM21B5C2A393JE02L" device="" value="0.1uF"/>
 <part name="SUPPLY7" library="supply2" library_urn="urn:adsk.eagle:library:372" deviceset="VSS" device=""/>
-<part name="SUPPLY8" library="supply2" library_urn="urn:adsk.eagle:library:372" deviceset="VSS" device=""/>
-<part name="+3V9" library="supply1" library_urn="urn:adsk.eagle:library:371" deviceset="+3V3" device=""/>
 <part name="C9" library="GCM21B5C2A393JE02L" deviceset="GCM21B5C2A393JE02L" device="" value="22uF"/>
 <part name="C4" library="GCM21B5C2A393JE02L" deviceset="GCM21B5C2A393JE02L" device="" value="10uF"/>
@@
 </instance>
 <instance part="C5" gate="G$1" x="-370.459" y="-2.667" smashed="yes">
-<attribute name="NAME" x="-368.935" y="-2.286" size="1.778" layer="95"/>
+<attribute name="NAME" x="-363.855" y="2.794" size="1.778" layer="95"/>
 <attribute name="VALUE" x="-368.935" y="-7.366" size="1.778" layer="96"/>
 </instance>
@@
 <attribute name="VALUE" x="-287.02" y="195.58" size="1.778" layer="96"/>
 </instance>
-<instance part="IC3" gate="G$1" x="-112.395" y="-10" smashed="yes">
-<attribute name="NAME" x="-104.775" y="-1.745" size="1.778" layer="95" align="center-left"/>
-<attribute name="VALUE" x="-105.41" y="-4.285" size="1.778" layer="96" align="center-left"/>
-</instance>
-<instance part="R1" gate="G$1" x="-135.255" y="-30.48" smashed="yes">
-<attribute name="NAME" x="-139.065" y="-28.9814" size="1.778" layer="95"/>
-<attribute name="VALUE" x="-139.065" y="-33.782" size="1.778" layer="96"/>
-</instance>
-<instance part="R6" gate="G$1" x="-130.175" y="-20.32" smashed="yes" rot="R90">
-<attribute name="NAME" x="-131.6736" y="-24.13" size="1.778" layer="95" rot="R90"/>
-<attribute name="VALUE" x="-126.873" y="-24.13" size="1.778" layer="96" rot="R90"/>
-</instance>
-<instance part="C1" gate="G$1" x="-98.425" y="4.445" smashed="yes" rot="R180">
-<attribute name="NAME" x="-99.949" y="4.064" size="1.778" layer="95" rot="R180"/>
-<attribute name="VALUE" x="-99.949" y="9.144" size="1.778" layer="96" rot="R180"/>
-</instance>
 <instance part="GND20" gate="1" x="-200.66" y="-36.83" smashed="yes">
 <attribute name="VALUE" x="-203.2" y="-39.37" size="1.778" layer="96"/>
 </instance>
-<instance part="GND21" gate="1" x="-124.46" y="-19.05" smashed="yes">
-<attribute name="VALUE" x="-127" y="-21.59" size="1.778" layer="96"/>
-</instance>
-<instance part="C3" gate="G$1" x="-131.445" y="0.3175" smashed="yes" rot="R270">
-<attribute name="NAME" x="-131.064" y="-1.2065" size="1.778" layer="95" rot="R270"/>
-<attribute name="VALUE" x="-136.144" y="-1.2065" size="1.778" layer="96" rot="R270"/>
-</instance>
 <instance part="SUPPLY7" gate="G$1" x="-187.96" y="-5.08" smashed="yes" rot="R180">
 <attribute name="VALUE" x="-186.055" y="-0.381" size="1.778" layer="96"/>
-</instance>
-<instance part="SUPPLY8" gate="G$1" x="-132.08" y="12.7" smashed="yes" rot="R180">
-<attribute name="VALUE" x="-130.175" y="17.399" size="1.778" layer="96"/>
-</instance>
-<instance part="+3V9" gate="G$1" x="-71.12" y="-2.8575" smashed="yes">
-<attribute name="VALUE" x="-73.66" y="-7.9375" size="1.778" layer="96" rot="R90"/>
 </instance>
 <instance part="C9" gate="G$1" x="-270.383" y="-4.699" smashed="yes">
@@
 </segment>
 <segment>
-<pinref part="IC3" gate="G$1" pin="V-"/>
-<pinref part="GND21" gate="1" pin="GND"/>
-<wire x1="-112.395" y1="-12.54" x2="-124.46" y2="-12.54" width="0.1524" layer="91"/>
-<wire x1="-124.46" y1="-12.54" x2="-124.46" y2="-16.51" width="0.1524" layer="91"/>
-</segment>
-<segment>
 <pinref part="C8" gate="G$1" pin="2"/>
 <pinref part="GND3" gate="1" pin="GND"/>
@@
 <wire x1="-342.5825" y1="60.6425" x2="-342.5825" y2="66.04" width="0.1524" layer="91"/>
 <wire x1="-342.5825" y1="66.04" x2="-335.28" y2="66.04" width="0.1524" layer="91"/>
-</segment>
-<segment>
-<pinref part="C3" gate="G$1" pin="1"/>
-<pinref part="SUPPLY8" gate="G$1" pin="VSS"/>
-<wire x1="-131.445" y1="0.3175" x2="-131.445" y2="10.16" width="0.1524" layer="91"/>
-<wire x1="-131.445" y1="10.16" x2="-132.08" y2="10.16" width="0.1524" layer="91"/>
 </segment>
 </net>
@@
 <wire x1="-340.36" y1="205.74" x2="-325.12" y2="205.74" width="0.1524" layer="91"/>
 <wire x1="-325.12" y1="205.74" x2="-325.12" y2="207.9625" width="0.1524" layer="91"/>
-</segment>
-<segment>
-<pinref part="IC3" gate="G$1" pin="V+"/>
-<pinref part="+3V9" gate="G$1" pin="+3V3"/>
-<wire x1="-86.995" y1="-12.54" x2="-71.12" y2="-12.54" width="0.1524" layer="91"/>
-<wire x1="-71.12" y1="-12.54" x2="-71.12" y2="-5.3975" width="0.1524" layer="91"/>
 </segment>
 </net>
@@
 <wire x1="-144.78" y1="-38.735" x2="-144.78" y2="-30.48" width="0.1524" layer="91"/>
 <junction x="-144.78" y="-30.48"/>
-<pinref part="R1" gate="G$1" pin="1"/>
-<wire x1="-144.78" y1="-30.48" x2="-140.335" y2="-30.48" width="0.1524" layer="91"/>
 </segment>
 </net>
@@
 <label x="-256.54" y="48.26" size="1.778" layer="95"/>
 </segment>
+<segment>
+<pinref part="C5" gate="G$1" pin="1"/>
+<wire x1="-370.459" y1="-2.667" x2="-378.46" y2="-2.667" width="0.1524" layer="91"/>
+<wire x1="-378.46" y1="-2.667" x2="-378.46" y2="-2.54" width="0.1524" layer="91"/>
+<label x="-378.46" y="-2.54" size="1.778" layer="95"/>
+</segment>
 </net>
 <net name="N$19" class="0">
@@
 </segment>
 </net>
-<net name="N$20" class="0">
-<segment>
-<pinref part="R1" gate="G$1" pin="2"/>
-<pinref part="R6" gate="G$1" pin="1"/>
-<wire x1="-130.175" y1="-30.48" x2="-130.175" y2="-25.4" width="0.1524" layer="91"/>
-</segment>
-</net>
-<net name="N$7" class="0">
-<segment>
-<pinref part="R6" gate="G$1" pin="2"/>
-<pinref part="IC3" gate="G$1" pin="+IN"/>
-<wire x1="-130.175" y1="-15.24" x2="-130.175" y2="-10" width="0.1524" layer="91"/>
-<wire x1="-130.175" y1="-10" x2="-112.395" y2="-10" width="0.1524" layer="91"/>
-<pinref part="C1" gate="G$1" pin="2"/>
-<wire x1="-112.395" y1="-10" x2="-112.395" y2="4.445" width="0.1524" layer="91"/>
-<wire x1="-112.395" y1="4.445" x2="-111.125" y2="4.445" width="0.1524" layer="91"/>
-<junction x="-112.395" y="-10"/>
-<pinref part="C3" gate="G$1" pin="2"/>
-<wire x1="-131.445" y1="-12.3825" x2="-131.445" y2="-15.24" width="0.1524" layer="91"/>
-<wire x1="-131.445" y1="-15.24" x2="-130.175" y2="-15.24" width="0.1524" layer="91"/>
-<junction x="-130.175" y="-15.24"/>
-</segment>
-</net>
-<net name="N$16" class="0">
-<segment>
-<pinref part="IC3" gate="G$1" pin="OUT"/>
-<wire x1="-86.995" y1="-10" x2="-86.995" y2="-10.16" width="0.1524" layer="91"/>
-<wire x1="-86.995" y1="-10.16" x2="-80.264" y2="-10.16" width="0.1524" layer="91"/>
-<wire x1="-80.264" y1="-10.16" x2="-78.74" y2="-10.16" width="0.1524" layer="91"/>
-<wire x1="-78.74" y1="-10.16" x2="-78.74" y2="5.08" width="0.1524" layer="91"/>
-<pinref part="C1" gate="G$1" pin="1"/>
-<wire x1="-78.74" y1="5.08" x2="-95.885" y2="5.08" width="0.1524" layer="91"/>
-<wire x1="-95.885" y1="5.08" x2="-98.425" y2="4.445" width="0.1524" layer="91"/>
-<wire x1="-80.264" y1="-10.16" x2="-80.264" y2="-23.114" width="0.1524" layer="91"/>
-<wire x1="-80.264" y1="-23.114" x2="-121.92" y2="-23.114" width="0.1524" layer="91"/>
-<junction x="-80.264" y="-10.16"/>
-<pinref part="IC3" gate="G$1" pin="-IN"/>
-<wire x1="-112.395" y1="-15.08" x2="-121.92" y2="-15.08" width="0.1524" layer="91"/>
-<wire x1="-121.92" y1="-15.08" x2="-121.92" y2="-23.114" width="0.1524" layer="91"/>
-</segment>
-</net>
